File: Caffeinated-AFTONSPARV.kicad_sch (KiCad schematic)
At the start: 35 parts, among them J1 PWR, J2 LED, J3 TagConnect, J4 USB, Q1 AO3400A, Q2 AO3400A, Q3 AO3400A, SW1 SW_Push, U1 ESP32-C3-MINI-1-[H/N]4, U2 SY8201ABC

Commit message: Added JST SH 4P
Added JST SH 4P connector for UART flashing, to schematic and PCB, and rerouted traces and components to make that happen
Parts:
- J4: footprint Connector_PinSocket_1.00mm:PinSocket_1x04_P1.00mm_Vertical -> JST_SH_BM04B-SRSS-TB_LF__SN__KiCad:BM04B-SRSS-TB_LFSN_; symbol Connector_Generic:Conn_01x04 -> BM04B-SRSS-TB_LF__SN_:BM04B-SRSS-TB_LF__SN_; Manufacturer_Name (none) -> JST (JAPAN SOLDERLESS TERMINALS); Manufacturer_Part_Number (none) -> BM04B-SRSS-TB(LF)(SN); Mouser Part Number (none) -> N/A; Mouser Price/Stock (none) -> https://www.mouser.co.uk/ProductDetail/JST-Commercial/BM04B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; now fitted; now in the parts list
- renumbered C5 to C1, C5 to C10, C5 to C11, C22 to C2, C5 to C3, C5 to C4, C5 to C6, C5 to C7, C5 to C9
Connections:
- net GND: now also J4.3; no longer J4.1 (Pin_1)
- net USB-D+: now also J4.1; no longer J4.2 (Pin_2)
- net USB-D-: now also J4.2; no longer J4.3 (Pin_3)
- no-connect marks 5 -> 6
